File: hardware/cosmas/motors.kicad_sch (KiCad schematic)
At the start: 6 parts, among them J3 MOTORA, J4 MOTORB, J5 DRIVER-POWER, J6 MOTOR-CONTROL, J7 MOT_A, J8 MOT_A

Commit message: adds OBC PCB
Other:
- moved on the sheet: J3, J4, J5, J6, J7, J8
